File: Kicad/Sherie-top-acrylic/Sherie-top-acrylic.kicad_pcb (KiCad board)
At the start: 2 copper layers, 278.3 x 81.9 mm, 122 parts, among them J1 TYPE-C-31-M-12, SW1 SW_PUSH, SW10 SW_PUSH, SW11 SW_PUSH, SW12 SW_PUSH, SW13 SW_PUSH, SW14 SW_PUSH, SW15 SW_PUSH, SW16 SW_PUSH, SW17 SW_PUSH, SW18 SW_PUSH, SW19 SW_PUSH, SW2 SW_PUSH, SW20 SW_PUSH, SW21 SW_PUSH, SW22 SW_PUSH, SW23 SW_PUSH, SW24 SW_PUSH, SW25 SW_PUSH, SW26 SW_PUSH, SW27 SW_PUSH, SW28 SW_PUSH, SW29 SW_PUSH, SW3 SW_PUSH, SW30 SW_PUSH, SW31 SW_PUSH, SW32 SW_PUSH, SW33 SW_PUSH, SW34 SW_PUSH, SW35 SW_PUSH, SW36 SW_PUSH, SW37 SW_PUSH, SW38 SW_PUSH, SW39 SW_PUSH, SW4 SW_PUSH, SW40 SW_PUSH, SW41 SW_PUSH, SW42 SW_PUSH, SW43 SW_PUSH, SW44 SW_PUSH, SW45 SW_PUSH, SW46 SW_PUSH, SW47 SW_PUSH, SW5 SW_PUSH, SW6 SW_PUSH, SW7 SW_PUSH, SW8 SW_PUSH, SW9 SW_PUSH, U1 ATmega32U4-A, U2 TPD4E05U06DQAR, Y1 16MHz

Commit message: reamp対応など
Parts:
- removed C1: 1uF, Capacitor_SMD:C_0805_2012Metric
- removed C2, C3, C4: 0.1uF, Capacitor_SMD:C_0805_2012Metric
- removed C5: 10uF, Capacitor_SMD:C_0805_2012Metric
- removed C6, C7: 22pF, Capacitor_SMD:C_0805_2012Metric
- removed D1, D10, D11, D12, D13, D14, D15, D16, D17, D18, D19, D2, D20, D21, D22, D23, D24, D25, D26, D27, D28, D29, D3, D30, D31, D32, D33, D34, D35, D36, D37, D38, D39, D4, D40, D41, D42, D43, D44, D45, D46, D47, D5, D6, D7, D8, D9: D, kbd_Parts:Diode_TH_SMD_without_holes
- removed ESDD1: ESD5Z5V0, Diode_SMD:D_SOD-523
- removed F1: SMD0805-050-16V, Fuse:Fuse_1206_3216Metric
- removed FB1: GZ2012D601TF, Inductor_SMD:L_0805_2012Metric
- removed G***: LOGO, LOGO
- removed J1: TYPE-C-31-M-12, locallib:HRO-TYPE-C-31-M-12-Assembly
- removed LED1: Green, my_footprints:LED0805-RD_GREEN
- removed R1, R4: 10k, Resistor_SMD:R_0805_2012Metric
- removed R2, R3: 22, Resistor_SMD:R_0805_2012Metric
- removed R5, R6: 5.1k, Resistor_SMD:R_0805_2012Metric
- removed R7: 1k, Resistor_SMD:R_0805_2012Metric
- removed REF** (x4): M3_Spacer_hex, my_footprints:M3_Spacer_hex
- removed RESET0: RESET_SW, my_footprints:SMD_reset
- removed SW1, SW13, SW14, SW26, SW27, SW39: SW_PUSH, kbd_SW_Hole:SW_Hole_1.75u
- removed SW10, SW11, SW12, SW15, SW16, SW17, SW18, SW19, SW2, SW20, SW21, SW22, SW23, SW24, SW25, SW28, SW29, SW3, SW30, SW31, SW32, SW33, SW34, SW35, SW36, SW37, SW38, SW4, SW46, SW5, SW6, SW7, SW8, SW9: SW_PUSH, kbd_SW_Hole:SW_Hole_1u
- removed SW40, SW41, SW45, SW47: SW_PUSH, kbd_SW_Hole:SW_Hole_1.5u
- removed SW42, SW44: SW_PUSH, kbd_SW_Hole:SW_Hole_1.25u
- removed SW43: SW_PUSH, kbd_SW_Hole:SW_Hole_2.75u
- removed U1: ATmega32U4-A, Package_QFP:TQFP-44_10x10mm_P0.8mm
- removed U2: TPD4E05U06DQAR, acheron_Components:USON-10_2.5x1.0mm_P0.5mm
- removed Y1: 16MHz, Crystal:Crystal_SMD_3225-4Pin_3.2x2.5mm
Routing:
- net row1: track 651.4 -> 0.00 mm, vias 2 -> 0
- net row0: track 357.4 -> 0.00 mm, vias 2 -> 0
- net col0: track 345.7 -> 0.00 mm
- net GND: track 345.1 -> 0.00 mm, vias 90 -> 0
- net col2: track 343.9 -> 0.00 mm, vias 8 -> 0
- net row2: track 337.0 -> 0.00 mm
- net row3: track 317.4 -> 0.00 mm, vias 2 -> 0
- net col1: track 296.6 -> 0.00 mm, vias 6 -> 0
- net +5V: track 273.1 -> 0.00 mm, vias 10 -> 0
- net col3: track 269.0 -> 0.00 mm, vias 8 -> 0
- net col4: track 257.1 -> 0.00 mm, vias 8 -> 0
- net col5: track 221.0 -> 0.00 mm, vias 8 -> 0
- net col6: track 197.5 -> 0.00 mm, vias 10 -> 0
- net col7: track 183.9 -> 0.00 mm, vias 8 -> 0
- net col8: track 169.5 -> 0.00 mm, vias 8 -> 0
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- removed copper zone on B.Cu, net GND
- removed copper zone on F.Cu, net GND
Other:
- outline, holes or cut-outs redrawn
- board text removed: "Dear..."
- board text removed: "Sherie"
- board text removed: "Sherie v1.0"
- board text removed: "designed by Flora"
- board text removed: "v1.0"
